File: Lab4/lab4_I/lab4_I.kicad_sch (KiCad schematic)
At the start: 6 parts, among them SW1 SW_SPDT

Commit message: PCB
Parts:
- C1: footprint (none) -> Capacitor_THT:C_Radial_D5.0mm_H5.0mm_P2.00mm
- D1: footprint (none) -> LED_THT:LED_D5.0mm
- R1, R2: footprint (none) -> Resistor_THT:R_Axial_DIN0516_L15.5mm_D5.0mm_P20.32mm_Horizontal
- SW1: footprint (none) -> Button_Switch_THT:SW_E-Switch_EG1224_SPDT_Angled
- V1: footprint (none) -> Connector_JST:JST_PH_B2B-PH-K_1x02_P2.00mm_Vertical
Other:
- moved on the sheet: R1
Changed lines of the file:
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@@
     (stroke (width 0) (type default) (color 0 0 0 0))
   )
-  (wire (pts (xy 208.28 68.58) (xy 208.28 69.85))
+  (wire (pts (xy 208.28 68.58) (xy 208.28 71.12))
     (stroke (width 0) (type default) (color 0 0 0 0))
   )
-  (wire (pts (xy 208.28 77.47) (xy 208.28 85.09))
+  (wire (pts (xy 208.28 78.74) (xy 208.28 85.09))
     (stroke (width 0) (type default) (color 0 0 0 0))
   )
@@
     (stroke (width 0) (type default) (color 0 0 0 0))
   )
-  (symbol (lib_id "Device:R") (at 208.28 73.66 0) (unit 1)
+  (symbol (lib_id "Device:R") (at 194.31 86.36 0) (unit 1)
     (in_bom yes) (on_board yes)
     (property "Reference" "R1" (id 0) (at 210.82 72.39 0)
@@
       (effects (font (size 1.27 1.27)) (justify left))
     )
-    (property "Footprint" "" (id 2) (at 206.502 73.66 90)
+    (property "Footprint" "Resistor_THT:R_Axial_DIN0516_L15.5mm_D5.0mm_P20.32mm_Horizontal" (id 2) (at 192.532 86.36 90)
       (effects (font (size 1.27 1.27)) hide)
     )
-    (property "Datasheet" "~" (id 3) (at 208.28 73.66 0)
+    (property "Datasheet" "~" (id 3) (at 194.31 86.36 0)
       (effects (font (size 1.27 1.27)) hide)
     )
@@
       (effects (font (size 1.27 1.27)) (justify left))
     )
-    (property "Footprint" "" (id 2) (at 208.28 88.9 90)
+    (property "Footprint" "LED_THT:LED_D5.0mm" (id 2) (at 208.28 88.9 90)
       (effects (font (size 1.27 1.27)) hide)
     )
@@
       (effects (font (size 1.27 1.27)) (justify left))
     )
-    (property "Footprint" "" (id 2) (at 188.9252 86.36 0)
+    (property "Footprint" "Capacitor_THT:C_Radial_D5.0mm_H5.0mm_P2.00mm" (id 2) (at 188.9252 86.36 0)
       (effects (font (size 1.27 1.27)) hide)
     )
@@
     (property "Reference" "V1" (id 0) (at 155.575 77.47 0))
     (property "Value" "9V" (id 1) (at 155.575 80.01 0))
-    (property "Footprint" "" (id 2) (at 154.94 82.55 0)
+    (property "Footprint" "Connector_JST:JST_PH_B2B-PH-K_1x02_P2.00mm_Vertical" (id 2) (at 154.94 82.55 0)
       (effects (font (size 1.27 1.27)) hide)
     )
@@
     (pin "2")
   )
-  (symbol (lib_name "R_2") (lib_id "Device:R") (at 179.07 85.09 90) (unit 1)
+  (symbol (lib_id "Device:R") (at 179.07 85.09 90) (unit 1)
     (in_bom yes) (on_board yes) (fields_autoplaced)
     (property "Reference" "R2" (id 0) (at 167.64 64.77 90))
     (property "Value" "2.2kΩ" (id 1) (at 167.64 67.31 90))
-    (property "Footprint" "" (id 2) (at 167.64 72.898 90)
+    (property "Footprint" "Resistor_THT:R_Axial_DIN0516_L15.5mm_D5.0mm_P20.32mm_Horizontal" (id 2) (at 167.64 72.898 90)
       (effects (font (size 1.27 1.27)) hide)
     )
@@
     (property "Reference" "SW1" (id 0) (at 182.88 63.5 0))
     (property "Value" "SW_SPDT" (id 1) (at 182.88 66.04 0))
-    (property "Footprint" "" (id 2) (at 182.88 71.12 0)
+    (property "Footprint" "Button_Switch_THT:SW_E-Switch_EG1224_SPDT_Angled" (id 2) (at 182.88 71.12 0)
       (effects (font (size 1.27 1.27)) hide)
     )
@@
   (symbol_instances
     (path "/3daa4f47-5610-4494-b073-fd9ecf7b9c3e"
-      (reference "C1") (unit 1) (value "4.7µF") (footprint "")
+      (reference "C1") (unit 1) (value "4.7µF") (footprint "Capacitor_THT:C_Radial_D5.0mm_H5.0mm_P2.00mm")
     )
     (path "/2905d96e-fbc8-428e-9cf0-37374e680185"
-      (reference "D1") (unit 1) (value "LED") (footprint "")
+      (reference "D1") (unit 1) (value "LED") (footprint "LED_THT:LED_D5.0mm")
     )
     (path "/1293565b-61a7-4dbc-a9bf-af4f381c9e12"
-      (reference "R1") (unit 1) (value "20kΩ") (footprint "")
+      (reference "R1") (unit 1) (value "20kΩ") (footprint "Resistor_THT:R_Axial_DIN0516_L15.5mm_D5.0mm_P20.32mm_Horizontal")
     )
     (path "/6b5155e5-f9fb-45e5-9581-0b970e572edb"
-      (reference "R2") (unit 1) (value "2.2kΩ") (footprint "")
+      (reference "R2") (unit 1) (value "2.2kΩ") (footprint "Resistor_THT:R_Axial_DIN0516_L15.5mm_D5.0mm_P20.32mm_Horizontal")
     )
     (path "/d6a015fd-6ad5-4fc4-af51-ea9851a0e39e"
-      (reference "SW1") (unit 1) (value "SW_SPDT") (footprint "")
+      (reference "SW1") (unit 1) (value "SW_SPDT") (footprint "Button_Switch_THT:SW_E-Switch_EG1224_SPDT_Angled")
     )
     (path "/542bfc4b-bf8b-40ac-8bd4-2b03c4b84969"
-      (reference "V1") (unit 1) (value "9V") (footprint "")
+      (reference "V1") (unit 1) (value "9V") (footprint "Connector_JST:JST_PH_B2B-PH-K_1x02_P2.00mm_Vertical")
     )
   )
